File: pihat-breakout/isolated-i2c-dac.kicad_sch (KiCad schematic)
At the start: 9 parts, among them J4 Conn_01x02_Pin, J5 Conn_01x06_Pin, J6 Isolator_ISO1540_I2C, U2 B0505S-1WR2

Commit message: fix(0.1uF->100nF)
Parts:
- C25, C27: value 0.1µF -> 100nF
Changed lines of the file:
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@@
 			)
 		)
-		(property "Value" "0.1µF"
+		(property "Value" "100nF"
 			(at 97.282 63.5 90)
 			(effects
@@
 			)
 		)
-		(property "Value" "0.1µF"
+		(property "Value" "100nF"
 			(at 172.212 63.5 90)
 			(effects
